Commit message: basic gazebo launch file

File: x001_description/urdf/common_properties/common_inertials.xacro (robot description, xacro)
@@ -1,4 +1,12 @@
 <?xml version="1.0"?>
 <robot xmlns:xacro="http://www.ros.org/wiki/xacro">
+    <xacro:macro name="box_inertial" params="m l w h">
+        <inertial>
+            <mass value="${m}" />
+            <inertia ixx="${1/12 * m * (h*h + l*l)}" ixy="0.0" ixz="0.0"
+                iyy="${1/12 * m * (w*w + h*h)}"
+                iyz="0.0" izz="${1/12 * m * (w*w + l*l)}" />
+        </inertial>
+    </xacro:macro>
     <xacro:macro name="cylinder_inertial" params="m r l">
         <inertial>
@@ -9,6 +17,7 @@
     </xacro:macro>
     <xacro:macro name="solid_sphere_inertial" params="m r">
-        <mass value="${m}"/>
-        <inertia ixx="${2/3 * m * r * r}" ixy="0.0" ixz="0.0" iyy="${2/3 * m * r * r}" iyz="0.0" izz="${2/3 * m * r * r}"/>
+        <mass value="${m}" />
+        <inertia ixx="${2/3 * m * r * r}" ixy="0.0" ixz="0.0" iyy="${2/3 * m * r * r}" iyz="0.0"
+            izz="${2/3 * m * r * r}" />
     </xacro:macro>
 </robot>

File: x001_description/urdf/x001_core.xacro (robot description, xacro)
@@ -1,10 +1,11 @@
 <?xml version="1.0"?>
 <robot xmlns:xacro="http://www.ros.org/wiki/xacro">
-    <xacro:property name="base_length" value="0.4" />
+    <xacro:property name="base_length" value="0.6" />
     <xacro:property name="base_width" value="0.3" />
     <xacro:property name="base_height" value="0.15" />
-    <xacro:property name="wheel_radius" value="0.05" />
+    <xacro:property name="wheel_radius" value="0.1" />
     <xacro:property name="wheel_length" value="0.04" />
-    <xacro:property name="caster_radius" value="0.02" />
+    <xacro:property name="caster_radius" value="0.03" />
+    <xacro:property name="caster_mass" value="2" />
     <!-- BASE LINKS -->
     <link name="base_footprint" />
@@ -17,6 +18,12 @@
             <origin xyz="0 0 0" rpy="0.0 0.0 0.0" />
         </visual>
+        <collision>
+            <geometry>
+                <box size="${base_length} ${base_width} ${base_height}" />
+            </geometry>
+        </collision>
+        <xacro:box_inertial m="1.0" l="${base_length}" w="${base_width}" h="${base_height}" />
     </link>
-    <joint name="base_footprint_link_joint" type="fixed">
+    <joint name="base_footprint_to_link" type="fixed">
         <parent link="base_footprint" />
         <child link="base_link" />
@@ -40,5 +47,5 @@
             <xacro:cylinder_inertial m="0.1" r="${wheel_radius}" l="${wheel_length}" />
         </link>
-        <joint name="base_link_${prefix}_wheel" type="continuous">
+        <joint name="base_link_to_${prefix}_wheel" type="continuous">
             <parent link="base_link" />
             <child link="${prefix}_wheel" />
@@ -66,7 +73,7 @@
             <origin xyz="0.0 0.0 0.0" rpy="0.0 0.0 0.0" />
         </collision>
-        <xacro:solid_sphere_inertial m="0.1" r="${caster_radius}" />
+        <xacro:solid_sphere_inertial m="${caster_mass}" r="${caster_radius}" />
     </link>
-    <joint name="base_link_caster_wheel" type="fixed">
+    <joint name="base_link_to_caster_wheel" type="fixed">
         <parent link="base_link" />
         <child link="caster_wheel" />
