Commit message: correctly spawn bot, rviz2 still broken and struggling to add plugin

File: x001_description/urdf/x001.urdf.xacro (robot description, xacro)
@@ -4,3 +4,14 @@
     <xacro:include filename="common_properties/common_inertials.xacro" />
     <xacro:include filename="x001_core.xacro" />
+    <!-- <xacro:include filename="plugins/diff_drive.xacro" /> -->
+    <plugin
+        filename="gz-sim-diff-drive-system"
+        name="gz::sim::systems::DiffDrive">
+        <left_joint>base_left_wheel_joint</left_joint>
+        <right_joint>base_right_wheel_joint</right_joint>
+        <wheel_separation>1.2</wheel_separation>
+        <wheel_radius>0.4</wheel_radius>
+        <odom_publish_frequency>1</odom_publish_frequency>
+        <topic>cmd_vel</topic>
+    </plugin>
 </robot>

File: x001_description/urdf/x001_core.xacro (robot description, xacro)
@@ -25,5 +25,5 @@
         <xacro:box_inertial m="1.0" l="${base_length}" w="${base_width}" h="${base_height}" />
     </link>
-    <joint name="base_footprint_to_link" type="fixed">
+    <joint name="base_footprint_base_link_joint" type="fixed">
         <parent link="base_footprint" />
         <child link="base_link" />
@@ -47,5 +47,5 @@
             <xacro:cylinder_inertial m="0.1" r="${wheel_radius}" l="${wheel_length}" />
         </link>
-        <joint name="base_link_to_${prefix}_wheel" type="continuous">
+        <joint name="base_${prefix}_wheel_joint" type="continuous">
             <parent link="base_link" />
             <child link="${prefix}_wheel" />
@@ -75,5 +75,5 @@
         <xacro:solid_sphere_inertial m="${caster_mass}" r="${caster_radius}" />
     </link>
-    <joint name="base_link_to_caster_wheel" type="fixed">
+    <joint name="base_caster_wheel_joint" type="fixed">
         <parent link="base_link" />
         <child link="caster_wheel" />
